File: pcb/eagle/vixen-copy/vixen1.brd (EAGLE design)
At the start: 89.6 x 59.5 mm, 33 parts, among them CN1 EXPANSIONPORT-VIC20-EDGEEDGE, IC1 74HCT393N, IC2 74AC157N, IC3 74AC157N, IC4 74AC157N, IC5 74AC157N, IC6 74ALS11N, IC8 74132N, IC9 74LS00N, U1 TMS4416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

Commit message: add BLK5 to netlist
Connections:
- new net !BLK5: CN1.13
Changed lines of the file:
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@@
 <contactref element="CN1" pad="19"/>
+</signal>
+<signal name="!BLK5">
+<contactref element="CN1" pad="13"/>
 </signal>
 </signals>
