File: pcb/eagle/vixen-copy/vixen1.sch (EAGLE design)
At the start: 33 parts, among them CN1 EXPANSIONPORT-VIC20-EDGEEDGE, IC1 74HCT393N, IC2 74AC157N, IC3 74AC157N, IC4 74AC157N, IC5 74AC157N, IC6 74ALS11N, IC8 74132N, IC9 74LS00N, U1 TMS4416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

Commit message: add BLK5 to netlist
Connections:
- new net !BLK5: CN1.!BLK5
Changed lines of the file:
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@@
 <instance part="IC9" gate="D" x="10.16" y="96.52"/>
 <instance part="C1" gate="G$1" x="129.54" y="99.06"/>
-<instance part="C2" gate="G$1" x="152.4" y="124.46" rot="R180"/>
+<instance part="C2" gate="G$1" x="152.4" y="124.46" rot="MR180"/>
 <instance part="C3" gate="G$1" x="109.22" y="124.46" rot="MR0"/>
 <instance part="C5" gate="G$1" x="-5.08" y="-17.78"/>
@@
 </segment>
 </net>
+<net name="!BLK5" class="0">
+<segment>
+<pinref part="CN1" gate="G$1" pin="!BLK5"/>
+<wire x1="30.48" y1="38.1" x2="33.02" y2="38.1" width="0.1524" layer="91"/>
+<label x="33.02" y="38.1" size="1.27" layer="95" xref="yes"/>
+</segment>
+</net>
